File: hardware/servo-test-board/servo-test-board.kicad_sch (KiCad schematic)
At the start: 3 parts, among them M1 Motor_DC, U1 DRV8231ADSGR

Commit message: update board and schema
Parts:
- removed M1: Motor_DC, symbol Motor:Motor_DC
- R1: footprint (none) -> Resistor_SMD:R_0402_1005Metric
- U1: footprint WSON8_DSG_TEX -> open-servo-controller:DRV8231ADSGR
Connections:
- net M+: now reaches U1.6 (OUT1)
- net M-: now reaches U1.8 (OUT2)
Changed lines of the file:
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@@
   (junction (at 48.26 68.58) (diameter 0) (color 0 0 0 0)
-  )
-  (wire (pts (xy 93.98 34.29) (xy 93.98 39.37))
-    (stroke (width 0) (type default))
   )
   (wire (pts (xy 39.37 63.5) (xy 39.37 68.58))
@@
   )
   (wire (pts (xy 39.37 55.88) (xy 39.37 46.99))
-    (stroke (width 0) (type default))
-  )
-  (wire (pts (xy 93.98 26.67) (xy 104.14 26.67))
     (stroke (width 0) (type default))
   )
@@
     (stroke (width 0) (type default))
   )
-  (wire (pts (xy 93.98 31.75) (xy 93.98 26.67))
-    (stroke (width 0) (type default))
-  )
-  (wire (pts (xy 93.98 39.37) (xy 104.14 39.37))
-    (stroke (width 0) (type default))
-  )
   (wire (pts (xy 48.26 68.58) (xy 48.26 59.69))
     (stroke (width 0) (type default))
@@
   )
   (label "IN-" (at 48.26 34.29 0) (fields_autoplaced)
+    (effects (font (size 1.27 1.27)) (justify left bottom))
+  )
+  (label "M+" (at 93.98 31.75 0) (fields_autoplaced)
+    (effects (font (size 1.27 1.27)) (justify left bottom))
+  )
+  (label "M-" (at 93.98 34.29 0) (fields_autoplaced)
     (effects (font (size 1.27 1.27)) (justify left bottom))
   )
@@
       (effects (font (size 1.524 1.524)))
     )
-    (property "Footprint" "WSON8_DSG_TEX" (at 71.12 25.654 0)
+    (property "Footprint" "open-servo-controller:DRV8231ADSGR" (at 71.12 25.654 0)
       (effects (font (size 1.524 1.524)) hide)
     )
@@
       (effects (font (size 1.27 1.27)) (justify left))
     )
-    (property "Footprint" "" (at 41.148 59.69 90)
+    (property "Footprint" "Resistor_SMD:R_0402_1005Metric" (at 41.148 59.69 90)
       (effects (font (size 1.27 1.27)) hide)
     )
@@
         )
       )
-    )
-  )
-  (symbol (lib_id "Motor:Motor_DC") (at 104.14 31.75 0) (unit 1)
-    (in_bom yes) (on_board yes) (dnp no) (fields_autoplaced)
-    (property "Reference" "M1" (at 109.22 33.02 0)
-      (effects (font (size 1.27 1.27)) (justify left))
-    )
-    (property "Value" "Motor_DC" (at 109.22 35.56 0)
-      (effects (font (size 1.27 1.27)) (justify left))
-    )
-    (property "Footprint" "" (at 104.14 34.036 0)
-      (effects (font (size 1.27 1.27)) hide)
-    )
-    (property "Datasheet" "~" (at 104.14 34.036 0)
-      (effects (font (size 1.27 1.27)) hide)
-    )
-    (pin "1")
-    (pin "2")
-    (instances
-      (project "servo-test-board"
-        (path "/bce6e242-f764-4fc2-ba2e-0586275ad3f5"
-          (reference "M1") (unit 1)
-        )
-      )
