File: hardware/servo-dev-board/servo-dev-board.kicad_sch (KiCad schematic)
At the start: 39 parts, among them J1 Conn_01x04, J2 Conn_01x05, J3 Conn_01x04, J4 Conn_02x05_Odd_Even, SW1 SW_Push, SW2 SW_Push, U1 DRV8231ADSGR, U2 SSP7615-33DFR, U3 STM32F301K8Ux, Y1 16MHz 9pF

Commit message: design pcb
Parts:
- removed D1: SS34, Diode_SMD:D_SMA, symbol Diode:SS34
- removed H3, H4, H5, H6: MountingHole, MountingHole:MountingHole_2.2mm_M2_DIN965_Pad, symbol Mechanical:MountingHole
- added MH1, MH2, MH3, MH4: MountingHole_Pad_MP, MountingHole:MountingHole_2.2mm_M2_Pad_Via, symbol Mechanical:MountingHole_Pad_MP
- J2: value Conn_01x05 -> Conn_01x05_MountingPin; footprint Connector_JST:JST_SH_SM05B-SRSS-TB_1x05-1MP_P1.00mm_Horizontal -> Connector_JST:JST_ZH_B5B-ZR-SM4-TF_1x05-1MP_P1.50mm_Vertical; symbol Connector_Generic:Conn_01x05 -> Connector_Generic_MountingPin:Conn_01x05_MountingPin
- J3: value Conn_01x04 -> Conn_01x04_MountingPin; symbol Connector_Generic:Conn_01x04 -> Connector_Generic_MountingPin:Conn_01x04_MountingPin
- J4: renamed from J1; value Conn_01x04 -> Conn_01x04_MountingPin; symbol Connector_Generic:Conn_01x04 -> Connector_Generic_MountingPin:Conn_01x04_MountingPin
- renumbered USB1 to J1, J4 to J5
Connections:
- net VBUS is gone; now on net +5V: J1.1 (VBUS)
- net +3V3: now also U1.4 (VREF)
- net GND: now also J2.3 (Pin_3), J2.MP (MountPin), J3.MP (MountPin), J4.MP (MountPin), MH1.1 (MP), MH2.1 (MP), MH3.1 (MP), MH4.1 (MP); no longer J2.4 (Pin_4)
- net M1: now also J2.4 (Pin_4); no longer J2.1 (Pin_1)
- net M2: now also J2.5 (Pin_5); no longer J2.2 (Pin_2)
- net POT: now also J2.1 (Pin_1); no longer J2.5 (Pin_5)
- net UART1_RX: now also J4.1 (Pin_1), R1.1; no longer J4.3 (Pin_3), R4.1
- net UART1_TX: now also J4.3 (Pin_3), R4.1; no longer J4.1 (Pin_1), R1.1
- net VREF: now also J2.2 (Pin_2); no longer J2.3 (Pin_3), U1.4 (VREF)
- net OSC_IN renamed OSC-
- net OSC_OUT renamed OSC+
Other:
- note added: "M2 Screw Mounting Holes"
- moved on the sheet: CL1, CL2, Y1

Commit message: update servo-dev-board
Parts:
- added C11: 22uF, Capacitor_SMD:C_0603_1608Metric, symbol Device:C
- C1, C2, C3, C6, C7: LCSC (none) -> C1525
- C10, C4, C5: LCSC (none) -> C52923
- C8: LCSC (none) -> C19666
- C9: LCSC (none) -> C15195
- CL1, CL2: LCSC (none) -> C1547
- H1, H2: LCSC (none) -> C6332201
- J1: LCSC (none) -> C428495
- J2: LCSC (none) -> C265440
- J3, J4: LCSC (none) -> C160390
- J5: footprint Connector_PinSocket_1.27mm:PinSocket_2x05_P1.27mm_Vertical_SMD -> lib:IDC-TH_10P-P1.27-X1270WV-2X05A-6TV01; LCSC (none) -> C2962225
- L1: LCSC (none) -> C76883
- LED1: LCSC (none) -> C2286
- R1, R2, R3, R4, R6: value 10K -> 4K7; LCSC (none) -> C25792
- R5: LCSC (none) -> C25792
- R7: LCSC (none) -> C25768
- SW1, SW2: LCSC (none) -> C221895
- U1: footprint Package_SON:WSON-8-1EP_2x2mm_P0.5mm_EP0.9x1.6mm_ThermalVias -> Package_SON:WSON-8-1EP_2x2mm_P0.5mm_EP0.9x1.6mm; LCSC (none) -> C5139865
- U2: LCSC (none) -> C3011523
- U3: LCSC (none) -> C111684
- Y1: LCSC (none) -> C13738
Connections:
- net +5V: now also C11.2
- net GND: now also C11.1
Other:
- moved on the sheet: C1, R7, U1
