File: hardware/encoder-board/encoder-board.kicad_sch (KiCad schematic)
At the start: 10 parts, among them J1 Conn_01x04, U1 ITR1204SR10A_TR(BY), U2 ITR1204SR10A_TR(BY)

Commit message: Rename project from open-servo-controller to open-servo-core
- Update project name in README.md with new structure and status
- Update firmware directory path references in VSCode and Zed settings
- Rename firmware directory to match new project name
- Update KiCad library references in all hardware files
- Fix package name in Cargo.toml
- Update 3D model paths in footprints

🤖 Generated with [Claude Code](https://claude.ai/code)
Parts:
- U1, U2: symbol open-servo-controller:ITR1204SR10A_TR(BY) -> open-servo-core:ITR1204SR10A_TR(BY)
Changed lines of the file:
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@@
 	)
 	(symbol
-		(lib_id "open-servo-controller:ITR1204SR10A_TR(BY)")
+		(lib_id "open-servo-core:ITR1204SR10A_TR(BY)")
 		(at 41.91 50.8 0)
 		(unit 1)
@@
 	)
 	(symbol
-		(lib_id "open-servo-controller:ITR1204SR10A_TR(BY)")
+		(lib_id "open-servo-core:ITR1204SR10A_TR(BY)")
 		(at 41.91 99.06 0)
 		(unit 1)
