File: hardware/encoder-board/encoder-board.kicad_pcb (KiCad board)
At the start: 4 copper layers, 25 x 25 mm, 10 parts, among them J1 Conn_01x04, U1 ITR1204SR10A_TR(BY), U2 ITR1204SR10A_TR(BY)

Commit message: fix encoder board references
Parts:
- U1, U2: footprint open-servo-controller:OPTO-SMD-4_ITR1204SR10A -> open-servo-core:OPTO-SMD-4_ITR1204SR10A
Changed lines of the file:
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@@
 		)
 	)
-	(footprint "open-servo-controller:OPTO-SMD-4_ITR1204SR10A"
+	(footprint "open-servo-core:OPTO-SMD-4_ITR1204SR10A"
 		(layer "B.Cu")
 		(at 114 105)
@@
 		)
 		(embedded_fonts no)
-		(model "/Users/aaronqian/projects/electronics/open-servo-controller/hardware/common/3DModels/OPTO-SMD-4_ITR1204SR10A.step"
+		(model "/Users/aaron/projects/open-servo-core/hardware/common/3DModels/OPTO-SMD-4_ITR1204SR10A.step"
 			(offset
 				(xyz 0.000051 0.000025 0.6)
@@
 		)
 	)
-	(footprint "open-servo-controller:OPTO-SMD-4_ITR1204SR10A"
+	(footprint "open-servo-core:OPTO-SMD-4_ITR1204SR10A"
 		(layer "B.Cu")
 		(at 111 105)
@@
 		)
 		(embedded_fonts no)
-		(model "/Users/aaronqian/projects/electronics/open-servo-controller/hardware/common/3DModels/OPTO-SMD-4_ITR1204SR10A.step"
+		(model "/Users/aaron/projects/open-servo-core/hardware/common/3DModels/OPTO-SMD-4_ITR1204SR10A.step"
 			(offset
 				(xyz 0.000051 0.000025 0.6)
