File: hardware/motor-mount/motor-mount.kicad_pcb (KiCad board)
At the start: 2 copper layers, 15 x 17.8 mm, 3 parts, among them M1 Motor_DC

Commit message: Rename project from open-servo-controller to open-servo-core
- Update project name in README.md with new structure and status
- Update firmware directory path references in VSCode and Zed settings
- Rename firmware directory to match new project name
- Update KiCad library references in all hardware files
- Fix package name in Cargo.toml
- Update 3D model paths in footprints

🤖 Generated with [Claude Code](https://claude.ai/code)
Parts:
- M1: footprint open-servo-controller:SG90_Motor -> open-servo-core:SG90_Motor
Changed lines of the file:
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@@
     )
   )
-  (footprint "open-servo-controller:SG90_Motor" (layer "F.Cu")
+  (footprint "open-servo-core:SG90_Motor" (layer "F.Cu")
     (at 30.79 24.328)
     (property "Sheetfile" "motor-mount.kicad_sch")
