File: hardware/servo-dev-board-stm32f301/servo-dev-board.kicad_sch (KiCad schematic)
At the start: 39 parts, among them J1 USB_B_Micro, J2 Conn_01x05_MountingPin, J3 Conn_01x04_MountingPin, J4 Conn_01x04_MountingPin, J5 Conn_02x05_Odd_Even, SW1 SW_Push, SW2 SW_Push, U1 DRV8231ADSGR, U2 SSP7615-33DFR, U3 STM32F301K8Ux, Y1 16MHz 9pF

Commit message: update usb connector due to parts shortage
Parts:
- J1: footprint Connector_USB:USB_Micro-B_Amphenol_10103594-0001LF_Horizontal -> Connector_USB:USB_Micro-B_Amphenol_10118194-0001LF_Horizontal
Changed lines of the file:
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@@
 			)
 		)
-		(property "Footprint" "Connector_USB:USB_Micro-B_Amphenol_10103594-0001LF_Horizontal"
+		(property "Footprint" "Connector_USB:USB_Micro-B_Amphenol_10118194-0001LF_Horizontal"
 			(at 29.21 36.83 0)
 			(effects
