File: hardware/boards/encoder-board/encoder-board.kicad_pcb (KiCad board)
At the start: 4 copper layers, 25 x 25 mm, 10 parts, among them J1 Conn_01x04, U1 ITR1204SR10A_TR(BY), U2 ITR1204SR10A_TR(BY)

Commit message: re-organize shared folders
Parts:
- U1, U2: footprint open-servo-core:OPTO-SMD-4_ITR1204SR10A -> shared:OPTO-SMD-4_ITR1204SR10A
