File: hardware/boards/encoder-board/encoder-board.kicad_pcb (KiCad board)
At the start: 4 copper layers, 25 x 25 mm, 10 parts, among them J1 Conn_01x04, U1 ITR1204SR10A_TR(BY), U2 ITR1204SR10A_TR(BY)

Commit message: hw: encoder-board 3v3 redesign, kicad 10 resave, lcsc field cleanup
Parts:
- R1, R3: value 680 -> 33K
- R2, R4: value 390 -> 100
Connections:
- net +5V renamed +3V3
Other:
- board text added: "3V"
- board text removed: "5V"
