File: hardware/boards/encoder-board/encoder-board.kicad_sch (KiCad schematic)
At the start: 10 parts, among them J1 Conn_01x04, U1 ITR1204SR10A_TR(BY), U2 ITR1204SR10A_TR(BY)

Commit message: re-organize shared folders
Parts:
- U1, U2: footprint open-servo-controller:OPTO-SMD-4_ITR1204SR10A -> shared:OPTO-SMD-4_ITR1204SR10A; symbol open-servo-core:ITR1204SR10A_TR(BY) -> shared:ITR1204SR10A_TR(BY); LCSC Part (none) -> C475373
Changed lines of the file:
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@@
 	)
 	(symbol
-		(lib_id "open-servo-core:ITR1204SR10A_TR(BY)")
+		(lib_id "shared:ITR1204SR10A_TR(BY)")
 		(at 48.26 55.88 0)
 		(unit 1)
@@
 		(fields_autoplaced yes)
 		(property "Reference" "U1"
-			(at 48.26 44.45 0)
+			(at 48.26 46.99 0)
 			(effects
 				(font
@@
 			)
 		)
-		(property "Footprint" "open-servo-controller:OPTO-SMD-4_ITR1204SR10A"
+		(property "Footprint" "shared:OPTO-SMD-4_ITR1204SR10A"
 			(at 48.26 66.04 0)
 			(effects
@@
 		)
 		(property "LCSC" "C475373"
+			(at 48.26 46.99 0)
+			(effects
+				(font
+					(size 1.27 1.27)
+				)
+				(hide yes)
+			)
+		)
+		(property "LCSC Part" "C475373"
 			(at 48.26 46.99 0)
 			(effects
@@
 	)
 	(symbol
-		(lib_id "open-servo-core:ITR1204SR10A_TR(BY)")
+		(lib_id "shared:ITR1204SR10A_TR(BY)")
 		(at 109.22 55.88 0)
 		(unit 1)
@@
 		(fields_autoplaced yes)
 		(property "Reference" "U2"
-			(at 109.22 44.45 0)
+			(at 109.22 46.99 0)
 			(effects
 				(font
@@
 			)
 		)
-		(property "Footprint" "open-servo-controller:OPTO-SMD-4_ITR1204SR10A"
+		(property "Footprint" "shared:OPTO-SMD-4_ITR1204SR10A"
 			(at 109.22 66.04 0)
 			(effects
@@
 			(at 109.22 46.99 0)
 			(effects
+				(font
+					(size 1.27 1.27)
+				)
+				(hide yes)
+			)
+		)
+		(property "LCSC Part" "C475373"
+			(at 109.22 46.99 0)
+			(effects
