File: hardware/boards/encoder-board/encoder-board.kicad_sch (KiCad schematic)
At the start: 10 parts, among them J1 Conn_01x04, U1 ITR1204SR10A_TR(BY), U2 ITR1204SR10A_TR(BY)

Commit message: hw: encoder-board 3v3 redesign, kicad 10 resave, lcsc field cleanup
Parts:
- C1, C2: LCSC (none) -> C49678
- C3: LCSC (none) -> C15850
- R1, R3: value 680 -> 33K; LCSC C22548 -> C17633
- R2, R4: value 390 -> 100; LCSC C125923 -> C17408
- U1, U2: LCSC Part C475373 -> (none)
Connections:
- net +5V renamed +3V3
