File: hardware/boards/motor-mount/motor-mount.kicad_pcb (KiCad board)
At the start: 2 copper layers, 15 x 17.8 mm, 3 parts, among them M1 Motor_DC

Commit message: re-organize shared folders
Parts:
- M1: footprint open-servo-core:SG90_Motor -> shared:SG90_Motor
