File: hardware/boards/motor-mount/motor-mount.kicad_sch (KiCad schematic)
At the start: 3 parts, among them M1 Motor_DC

Commit message: re-organize shared folders
Parts:
- M1: footprint open-servo-core:SG90_Motor -> shared:SG90_Motor
Changed lines of the file:
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@@
 (kicad_sch
-	(version 20231120)
+	(version 20250114)
 	(generator "eeschema")
-	(generator_version "8.0")
+	(generator_version "9.0")
 	(paper "A4")
 	(junction
@@
 			)
 		)
-		(property "Footprint" "open-servo-core:SG90_Motor"
+		(property "Footprint" "shared:SG90_Motor"
 			(at 170.18 101.346 0)
 			(effects
@@
 		)
 	)
+	(embedded_fonts no)
 )
