File: hardware/boards/servo-dev-board-stm32f301/servo-dev-board.kicad_pcb (KiCad board)
At the start: 4 copper layers, 51.5 x 26.5 mm, 39 parts, among them J1 USB_B_Micro, J2 Conn_01x05_MountingPin, J3 Conn_01x04_MountingPin, J4 Conn_01x04_MountingPin, J5 Conn_02x05_Odd_Even, SW1 SW_Push, SW2 SW_Push, U1 DRV8231ADSGR, U2 SSP7615-33DFR, U3 STM32F301K8Ux, Y1 16MHz 9pF

Commit message: re-organize shared folders
Parts:
- removed U1: DRV8231ADSGR, Package_SON:WSON-8-1EP_2x2mm_P0.5mm_EP0.9x1.6mm
- added U4: DRV8231ADSG, Package_SON:WSON-8-1EP_2x2mm_P0.5mm_EP0.9x1.6mm, F.Cu at (125.8, 96.8)
- J5: footprint lib:IDC-TH_10P-P1.27-X1270WV-2X05A-6TV01 -> shared:IDC-TH_10P-P1.27-X1270WV-2X05A-6TV01
