File: hardware/boards/servo-dev-board-ch32v006/DIAGNOSTICS.kicad_sch (KiCad schematic)
At the start: 28 parts

Commit message: added MFPN properties
Parts:
- TP1, TP10, TP11, TP12, TP13, TP14, TP15, TP16, TP17, TP18, TP19, TP2, TP20, TP21, TP22, TP23, TP24, TP25, TP26, TP27, TP28, TP3, TP4, TP5, TP6, TP7, TP8, TP9: MFPN (none) -> RH-5015

Commit message: update board
Other:
- moved on the sheet: TP22
Changed lines of the file:
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@@
 	(wire
 		(pts
-			(xy 139.7 50.8) (xy 133.35 50.8)
+			(xy 133.35 52.07) (xy 139.7 52.07)
 		)
 		(stroke
@@
 	(hierarchical_label "MOT_A"
 		(shape passive)
-		(at 133.35 50.8 180)
+		(at 133.35 52.07 180)
 		(effects
 			(font
@@
 		(dnp no)
 		(fields_autoplaced yes)
-		(property "Reference" "#PWR046"
+		(property "Reference" "#PWR050"
 			(at 76.2 45.72 0)
 			(hide yes)
@@
 			(project "servo-dev-board-ch32v006"
 				(path "/6062e7d2-0c72-467e-b49c-6387ba053e09/279fdd48-5106-437c-982b-915097006b04"
-					(reference "#PWR046")
+					(reference "#PWR050")
 					(unit 1)
 				)
@@
 		(dnp no)
 		(fields_autoplaced yes)
-		(property "Reference" "#PWR047"
+		(property "Reference" "#PWR051"
 			(at 76.2 91.44 0)
 			(hide yes)
@@
 			(project "servo-dev-board-ch32v006"
 				(path "/6062e7d2-0c72-467e-b49c-6387ba053e09/279fdd48-5106-437c-982b-915097006b04"
-					(reference "#PWR047")
+					(reference "#PWR051")
 					(unit 1)
 				)
@@
 	(symbol
 		(lib_id "Connector:TestPoint_Probe")
-		(at 139.7 50.8 270)
+		(at 139.7 52.07 270)
 		(mirror x)
 		(unit 1)
@@
 		(fields_autoplaced yes)
 		(property "Reference" "TP22"
-			(at 143.51 49.2124 90)
+			(at 143.51 50.4824 90)
 			(show_name no)
 			(do_not_autoplace no)
@@
 		)
 		(property "Value" "TestPoint_Probe"
-			(at 140.0176 46.99 0)
+			(at 140.0176 48.26 0)
 			(hide yes)
 			(show_name no)
@@
 		)
 		(property "Footprint" "TestPoint:TestPoint_Keystone_5015_Micro_Mini"
-			(at 139.7 45.72 0)
+			(at 139.7 46.99 0)
 			(hide yes)
 			(show_name no)
@@
 		)
 		(property "Datasheet" ""
-			(at 139.7 45.72 0)
+			(at 139.7 46.99 0)
 			(hide yes)
 			(show_name no)
@@
 		)
 		(property "Description" "test point (alternative probe-style design)"
-			(at 139.7 50.8 0)
+			(at 139.7 52.07 0)
 			(hide yes)
 			(show_name no)
@@
 		)
 		(property "LCSC" "C5199798"
-			(at 139.7 50.8 0)
+			(at 139.7 52.07 0)
 			(hide yes)
 			(show_name no)
@@
 		)
 		(property "MFPN" "RH-5015"
-			(at 139.7 50.8 0)
+			(at 139.7 52.07 0)
 			(hide yes)
 			(show_name no)
@@
 		)
 		(property "JLC Type" "Extended"
-			(at 139.7 50.8 0)
+			(at 139.7 52.07 0)
 			(hide yes)
 			(show_name no)
@@
 		(dnp no)
 		(fields_autoplaced yes)
-		(property "Reference" "#PWR048"
+		(property "Reference" "#PWR052"
 			(at 127 60.96 0)
 			(hide yes)
@@
 			(project "servo-dev-board-ch32v006"
 				(path "/6062e7d2-0c72-467e-b49c-6387ba053e09/279fdd48-5106-437c-982b-915097006b04"
-					(reference "#PWR048")
+					(reference "#PWR052")
 					(unit 1)
 				)
@@
 		(dnp no)
 		(fields_autoplaced yes)
-		(property "Reference" "#PWR045"
+		(property "Reference" "#PWR049"
 			(at 46.99 91.44 0)
 			(hide yes)
@@
 			(project "servo-dev-board-ch32v006"
 				(path "/6062e7d2-0c72-467e-b49c-6387ba053e09/279fdd48-5106-437c-982b-915097006b04"
-					(reference "#PWR045")
+					(reference "#PWR049")
 					(unit 1)
 				)
@@
 		(dnp no)
 		(fields_autoplaced yes)
-		(property "Reference" "#PWR044"
+		(property "Reference" "#PWR048"
 			(at 46.99 45.72 0)
 			(hide yes)
@@
 			(project "servo-dev-board-ch32v006"
 				(path "/6062e7d2-0c72-467e-b49c-6387ba053e09/279fdd48-5106-437c-982b-915097006b04"
-					(reference "#PWR044")
+					(reference "#PWR048")
 					(unit 1)
 				)
