File: hardware/boards/osc-dev-m007/osc-dev-m007.kicad_sch (KiCad schematic)
At the start: 2 parts, among them Q1 SIL3724A-TP

Commit message: hw: design osc-dev-m007 schematics
Parts:
- removed D1: XL-1010RGBC-WS2812B, shared:LED_XL-1010RGBC-WS2812B_1x1mm, symbol shared:XL-1010RGBC-WS2812B
- removed Q1: SIL3724A-TP, Package_TO_SOT_SMD:SOT-23-6, symbol shared:SIL3724A-TP
- added H101, H102, H103, H104: MountingHole_Pad_MP, MountingHole:MountingHole_2.2mm_M2_ISO7380_Pad, symbol Mechanical:MountingHole_Pad
Connections:
- new net GND: H101.1, H102.1, H103.1, H104.1
Other:
- added sheet BRIDGE (bridge.kicad_sch)
- added sheet BUS (bus.kicad_sch)
- added sheet POWER (power.kicad_sch)
- added sheet SENSORS (sensors.kicad_sch)
- added sheet TESTPOINTS (testpoints.kicad_sch)
- sheet MCU ports: added BUS, ENC, GATE_AH, GATE_AL, GATE_BH, GATE_BL, GATE_CH, GATE_CL, ISNS-, ISNS1+, ISNS2+, NTC, POS, VSNA, VSNB, VSNC; removed none
