File: hardware/boards/osc-dev-m007/bridge.kicad_sch (KiCad schematic)
At the start: 3 parts, among them J301 BDC, J302 BLDC

Commit message: hw: design osc-dev-m007 pcb
Parts:
- removed J301: BDC, Connector_PinHeader_2.54mm:PinHeader_1x02_P2.54mm_Vertical, symbol Connector_Generic:Conn_01x02
- removed J302: BLDC, Connector_PinHeader_2.54mm:PinHeader_1x03_P2.54mm_Vertical, symbol Connector_Generic:Conn_01x03
- added J301: BLDC/BDC(A+B), shared:CONN-TH_3P-P3.50_KF350-3.5-3P, symbol Connector:Screw_Terminal_01x03
Connections:
- net PH_A: now also J301.1 (Pin_1)
- net PH_B: now also J301.2 (Pin_2)
- net PH_C: now also J301.3 (Pin_3)
