File: hardware/boards/osc-dev-m007/bus.kicad_sch (KiCad schematic)
At the start: 7 parts, among them J1101 PIN-1-3P, J1102 PIN-1-3P, J1103 JST-PH-V, J1104 JST-PH-V

Commit message: hw: design osc-dev-m007 pcb
Parts:
- removed J1101, J1102: PIN-1-3P, Connector_PinHeader_2.54mm:PinHeader_1x03_P2.54mm_Vertical, symbol Connector_Generic:Conn_01x03
- renumbered J1103 to J1101, J1104 to J1102
Other:
- note removed: "OSC TTL CONNECTOR 2.54mm 3P VERTICAL"
- moved on the sheet: J1101, J1102

Commit message: hw: add osc-sg90-m007 renders to readme
Parts:
- R1101: value 33Ω -> 33
- R1102: value 10kΩ -> 10k
Changed lines of the file:
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@@
 			)
 		)
-		(property "Value" "33Ω"
+		(property "Value" "33"
 			(at 36.83 64.516 90)
 			(show_name no)
@@
 			)
 		)
-		(property "Value" "10kΩ"
+		(property "Value" "10k"
 			(at 46.99 58.4199 0)
 			(show_name no)

Commit message: hw: swap dev-m007 parts to in-stock equivalents
Parts:
- R1102: LCSC C17414 -> C2907219; MFPN 0805W8F1002T5E -> FRC0805F1002TS
Changed lines of the file:
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@@
 			)
 		)
-		(property "Datasheet" "https://www.lcsc.com/product-detail/C17414.html"
+		(property "Datasheet" "https://www.lcsc.com/product-detail/C2907219.html"
 			(at 44.45 57.15 0)
 			(hide yes)
@@
 			)
 		)
-		(property "LCSC" "C17414"
+		(property "LCSC" "C2907219"
 			(at 46.99 55.8799 0)
 			(hide yes)
@@
 			)
 		)
-		(property "MFPN" "0805W8F1002T5E"
+		(property "MFPN" "FRC0805F1002TS"
 			(at 46.99 55.8799 0)
 			(hide yes)
