File: hardware/boards/osc-dev-m007/mcu.kicad_sch (KiCad schematic)
At the start: 7 parts, among them U1 CH32M007E8U7

Commit message: hw: design osc-dev-m007 schematics
Parts:
- removed C1: 2.2uF, symbol Device:C_Small
- removed C2, C4: 0.1uF, symbol Device:C_Small
- removed C3, C5: 10uF, symbol Device:C_Small
- removed R1: 0, symbol Device:R_Small
- added C201, C202: 2.2uF, Capacitor_SMD:C_0805_2012Metric_Pad1.18x1.45mm_HandSolder, symbol Device:C_Small
- added C203, C206, C209, C210: 0.1uF, Capacitor_SMD:C_0805_2012Metric_Pad1.18x1.45mm_HandSolder, symbol Device:C_Small
- added C204, C205, C208: 10uF, Capacitor_SMD:C_1206_3216Metric_Pad1.33x1.80mm_HandSolder, symbol Device:C_Small
- added C207: 1uF, Capacitor_SMD:C_0805_2012Metric_Pad1.18x1.45mm_HandSolder, symbol Device:C_Small
- added D201: STAT, shared:LED_XL-1010RGBC-WS2812B_1x1mm, symbol shared:XL-1010RGBC-WS2812B
- added J201: PROG, Connector_PinHeader_2.54mm:PinHeader_1x05_P2.54mm_Vertical, symbol Connector_Generic:Conn_01x05
- added R201: 0Ω, Resistor_SMD:R_0805_2012Metric_Pad1.20x1.40mm_HandSolder, symbol Device:R_Small
- added R202: 10KΩ, Resistor_SMD:R_0805_2012Metric_Pad1.20x1.40mm_HandSolder, symbol Device:R_Small
- added R203: 100Ω, Resistor_SMD:R_0805_2012Metric_Pad1.20x1.40mm_HandSolder, symbol Device:R_Small
- added SW201: RESET, shared:SW_SPST_TS-1088R_3.9x3.0mm, symbol shared:TS-1088R-02026
- U201: renamed from U1; JLC_Basic (none) -> no; MFPN (none) -> CH32M007E8U7
Connections:
- net +5V: now also C206.1, C207.1, C208.1, C210.1, D201.2 (VDD), R202.1
- net GND: now also C201.2, C202.2, C203.2, C204.2, C205.2, C207.2, C209.1, C210.2, D201.3 (VSS), J201.2 (Pin_2), J201.4 (Pin_4), SW201.1
- net LED: now also R203.1
- net SWDIO: now also J201.1 (Pin_1)
- net VHREG: now also C201.1, C202.1, R201.1
- net VSYS: now also C203.1, C204.1, C205.1, R201.2
- net nRST: now also C209.2, J201.5 (Pin_5), R202.2, SW201.2
- new net: D201.4 (DIN), R203.2
- new net: C206.2, C208.2
- new net VPROG: J201.3 (Pin_3)
- no-connect marks 0 -> 1
Other:
- moved on the sheet: U201

Commit message: hw: design osc-dev-m007 pcb
Connections:
- net GND: now also C206.2, C208.2
Changed lines of the file:
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@@
+	)
+	(junction
+		(at 49.53 93.98)
+		(diameter 0)
+		(color 0 0 0 0)
 	)
 	(junction
@@
 	(wire
 		(pts
+			(xy 27.94 93.98) (xy 49.53 93.98)
+		)
+		(stroke
+			(width 0)
+			(type default)
+		)
+	)
+	(wire
+		(pts
 			(xy 147.32 135.89) (xy 147.32 134.62)
 		)
@@
 	(wire
 		(pts
-			(xy 27.94 93.98) (xy 69.85 93.98)
-		)
-		(stroke
-			(width 0)
-			(type default)
-		)
-	)
-	(wire
-		(pts
 			(xy 38.1 60.96) (xy 49.53 60.96)
 		)
@@
 	(wire
 		(pts
+			(xy 49.53 93.98) (xy 69.85 93.98)
+		)
+		(stroke
+			(width 0)
+			(type default)
+		)
+	)
+	(wire
+		(pts
 			(xy 49.53 45.72) (xy 59.69 45.72)
 		)
@@
 	(wire
 		(pts
-			(xy 49.53 90.17) (xy 49.53 95.25)
+			(xy 49.53 90.17) (xy 49.53 93.98)
 		)
 		(stroke
@@
 		)
 		(stroke
+			(width 0)
+			(type default)
+		)
+	)
+	(wire
+		(pts
+			(xy 49.53 93.98) (xy 49.53 95.25)
+		)
+		(stroke

Commit message: hw: add osc-sg90-m007 renders to readme
Parts:
- R201: value 0Ω -> 0
- R202: value 10KΩ -> 10k
- R203: value 100Ω -> 100
Changed lines of the file:
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@@
 			)
 		)
-		(property "Value" "0Ω"
+		(property "Value" "0"
 			(at 43.18 47.625 90)
 			(show_name no)
@@
 			)
 		)
-		(property "Value" "100Ω"
+		(property "Value" "100"
 			(at 90.17 130.302 90)
 			(show_name no)
@@
 			)
 		)
-		(property "Value" "10KΩ"
+		(property "Value" "10k"
 			(at 48.006 124.714 0)
 			(show_name no)

Commit message: hw: swap dev-m007 parts to in-stock equivalents
Parts:
- J201: now left out of the parts list
- R202: LCSC C17414 -> C2907219; MFPN 0805W8F1002T5E -> FRC0805F1002TS
Changed lines of the file:
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@@
 			)
 		)
-		(property "Datasheet" "https://www.lcsc.com/product-detail/C17414.html"
+		(property "Datasheet" "https://www.lcsc.com/product-detail/C2907219.html"
 			(at 46.99 124.46 0)
 			(hide yes)
@@
 			)
 		)
-		(property "MFPN" "0805W8F1002T5E"
+		(property "MFPN" "FRC0805F1002TS"
 			(at 46.99 124.46 0)
 			(hide yes)
@@
 			)
 		)
-		(property "LCSC" "C17414"
+		(property "LCSC" "C2907219"
 			(at 46.99 124.46 0)
 			(hide yes)
@@
 		(body_style 1)
 		(exclude_from_sim no)
-		(in_bom yes)
+		(in_bom no)
 		(on_board yes)
 		(in_pos_files yes)
