File: hardware/boards/osc-dev-m007/sensors.kicad_sch (KiCad schematic)
At the start: 11 parts, among them J1001 NTC_EXT, J1002 ENC, J1003 POT

Commit message: hw: add osc-sg90-m007 renders to readme
Parts:
- C1002, C1003: value 0.1µF -> 0.1uF
- R1001: value 10kΩ -> 10k
- R1002, R1003: value 4.7kΩ -> 4.7k
- TH1001: value 10kΩ 3950K -> 10k 3950K
Changed lines of the file:
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@@
 			)
 		)
-		(property "Value" "0.1µF"
+		(property "Value" "0.1uF"
 			(at 102.362 50.8 0)
 			(show_name no)
@@
 			)
 		)
-		(property "Value" "0.1µF"
+		(property "Value" "0.1uF"
 			(at 123.952 102.87 0)
 			(show_name no)
@@
 			)
 		)
-		(property "Value" "10kΩ 3950K"
+		(property "Value" "10k 3950K"
 			(at 116.84 105.41 0)
 			(show_name no)
@@
 			)
 		)
-		(property "Value" "10kΩ"
+		(property "Value" "10k"
 			(at 80.01 88.9 0)
 			(show_name no)
@@
 			)
 		)
-		(property "Value" "4.7kΩ"
+		(property "Value" "4.7k"
 			(at 88.9 46.99 90)
 			(show_name no)
@@
 			)
 		)
-		(property "Value" "4.7kΩ"
+		(property "Value" "4.7k"
 			(at 87.63 148.59 90)
 			(show_name no)

Commit message: hw: swap dev-m007 parts to in-stock equivalents
Parts:
- C1001: LCSC C46653 -> C94121; MFPN CL21B102KBCNNNC -> CC0805KRX7R9BB102
- J1001, J1002, J1003, JP1001: now left out of the parts list
- R1001: LCSC C17414 -> C2907219; MFPN 0805W8F1002T5E -> FRC0805F1002TS
- TH1001: LCSC C95968 -> C49247662; MFPN SDNT2012X103F3950FTF -> HNTC0805-103F3950FB
Changed lines of the file:
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@@
 		(body_style 1)
 		(exclude_from_sim no)
-		(in_bom yes)
+		(in_bom no)
 		(on_board yes)
 		(in_pos_files yes)
@@
 		(body_style 1)
 		(exclude_from_sim no)
-		(in_bom yes)
+		(in_bom no)
 		(on_board yes)
 		(in_pos_files yes)
@@
 		(body_style 1)
 		(exclude_from_sim no)
-		(in_bom yes)
+		(in_bom no)
 		(on_board yes)
 		(in_pos_files yes)
@@
 			)
 		)
-		(property "Datasheet" "https://www.lcsc.com/product-detail/C95968.html"
+		(property "Datasheet" "https://www.lcsc.com/product-detail/C49247662.html"
 			(at 102.87 104.14 0)
 			(hide yes)
@@
 			)
 		)
-		(property "Description" "NTC 10kΩ 3950K -55℃~+125℃"
+		(property "Description" "NTC 10k 3950K -40C~+125C"
 			(at 102.87 104.14 0)
 			(hide yes)
@@
 			)
 		)
-		(property "LCSC" "C95968"
+		(property "LCSC" "C49247662"
 			(at 99.06 102.8699 0)
 			(hide yes)
@@
 			)
 		)
-		(property "MFPN" "SDNT2012X103F3950FTF"
+		(property "MFPN" "HNTC0805-103F3950FB"
 			(at 99.06 102.8699 0)
 			(hide yes)
@@
 			)
 		)
-		(property "Datasheet" "https://www.lcsc.com/product-detail/C17414.html"
+		(property "Datasheet" "https://www.lcsc.com/product-detail/C2907219.html"
 			(at 82.55 87.63 0)
 			(hide yes)
@@
 			)
 		)
-		(property "LCSC" "C17414"
+		(property "LCSC" "C2907219"
 			(at 86.614 85.852 0)
 			(hide yes)
@@
 			)
 		)
-		(property "MFPN" "0805W8F1002T5E"
+		(property "MFPN" "FRC0805F1002TS"
 			(at 86.614 85.852 0)
 			(hide yes)
@@
 			)
 		)
-		(property "Datasheet" "https://www.lcsc.com/product-detail/C46653.html"
+		(property "Datasheet" "https://www.lcsc.com/product-detail/C94121.html"
 			(at 79.29 130.25 0)
 			(hide yes)
@@
 			)
 		)
-		(property "LCSC" "C46653"
+		(property "LCSC" "C94121"
 			(at 91.694 151.384 0)
 			(hide yes)
@@
 			)
 		)
-		(property "MFPN" "CL21B102KBCNNNC"
+		(property "MFPN" "CC0805KRX7R9BB102"
 			(at 91.694 151.384 0)
 			(hide yes)
@@
 		(body_style 1)
 		(exclude_from_sim no)
-		(in_bom yes)
+		(in_bom no)
 		(on_board yes)
 		(in_pos_files yes)
