File: hardware/boards/osc-dev-m007/shunt.kicad_sch (KiCad schematic)
At the start: 6 parts

Commit message: hw: swap dev-m007 parts to in-stock equivalents
Parts:
- C501: LCSC C46653 -> C94121; MFPN CL21B102KBCNNNC -> CC0805KRX7R9BB102
- R_SH501: LCSC C859920 -> C49164946; MFPN RL1206FR-7W0R075L -> JER1206F1R075
- R_SH502: LCSC C859925 -> C2683383; MFPN RL1206FR-7W0R15L -> RLH12FTCR150
Changed lines of the file:
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@@
 			)
 		)
-		(property "Datasheet" "https://www.lcsc.com/product-detail/C859920.html"
+		(property "Datasheet" "https://www.lcsc.com/product-detail/C49164946.html"
 			(at 41.91 50.8 0)
 			(hide yes)
@@
 			)
 		)
-		(property "Description" "Current sense resistor 75mΩ ±1% 0.5W 1206"
+		(property "Description" "Current sense resistor 75mOhm 1% 1W 1206"
 			(at 41.91 50.8 0)
 			(hide yes)
@@
 			)
 		)
-		(property "MFPN" "RL1206FR-7W0R075L"
+		(property "MFPN" "JER1206F1R075"
 			(at 41.91 50.8 0)
 			(hide yes)
@@
 			)
 		)
-		(property "LCSC" "C859920"
+		(property "LCSC" "C49164946"
 			(at 41.91 50.8 0)
 			(hide yes)
@@
 			)
 		)
-		(property "Datasheet" "https://www.lcsc.com/product-detail/C46653.html"
+		(property "Datasheet" "https://www.lcsc.com/product-detail/C94121.html"
 			(at 124.46 60.96 0)
 			(hide yes)
@@
 			)
 		)
-		(property "MFPN" "CL21B102KBCNNNC"
+		(property "MFPN" "CC0805KRX7R9BB102"
 			(at 124.46 60.96 0)
 			(hide yes)
@@
 			)
 		)
-		(property "LCSC" "C46653"
+		(property "LCSC" "C94121"
 			(at 124.46 60.96 0)
 			(hide yes)
@@
 			)
 		)
-		(property "Datasheet" "https://www.lcsc.com/product-detail/C859925.html"
+		(property "Datasheet" "https://www.lcsc.com/product-detail/C2683383.html"
 			(at 55.88 50.8 0)
 			(hide yes)
@@
 			)
 		)
-		(property "Description" "Current sense resistor 150mΩ ±1% 0.5W 1206"
+		(property "Description" "Current sense resistor 150mOhm 1% 1W 1206"
 			(at 55.88 50.8 0)
 			(hide yes)
@@
 			)
 		)
-		(property "MFPN" "RL1206FR-7W0R15L"
+		(property "MFPN" "RLH12FTCR150"
 			(at 55.88 50.8 0)
 			(hide yes)
@@
 			)
 		)
-		(property "LCSC" "C859925"
+		(property "LCSC" "C2683383"
 			(at 55.88 50.8 0)
 			(hide yes)
