File: hardware/boards/osc-sg90-m007/osc-sg90-m007.kicad_pcb (KiCad board)
At the start: 6 copper layers, 12.1 x 9.6 mm, 32 parts, among them J1 TTL, J2 Motor, J3 PROG, J4 POT, Q1 MCMNP2065A-TP, Q2 MCMNP2065A-TP, U1 CH32M007E8U7

Commit message: hw: add osc-sg90-m007 renders to readme
Parts:
- C1, C3: value 10µF -> 10uF
- C2, C8: value 0.1µF -> 0.1uF
- C4: value 2.2µF -> 2.2uF
- C5: value 0.1µF 25V -> 0.1uF 25V
- R1, R2, R5, R6: value 100K -> 100k
- R11: value 4.7kΩ -> 4.7k
- R12, R4, R8: value 10kΩ -> 10k
- R13: value 33Ω -> 33
- R3, R7: value 20kΩ -> 20k
Changed lines of the file:
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@@
 			)
 		)
-		(property "Value" "20kΩ"
+		(property "Value" "20k"
 			(at 0 1.17 180)
 			(layer "F.Fab")
@@
 			)
 		)
-		(property "Value" "4.7kΩ"
+		(property "Value" "4.7k"
 			(at 0 1.17 90)
 			(layer "F.Fab")
@@
 			)
 		)
-		(property "Value" "100K"
+		(property "Value" "100k"
 			(at 0 1.169999 127.235)
 			(layer "F.Fab")
@@
 			)
 		)
-		(property "Value" "33Ω"
+		(property "Value" "33"
 			(at 0 1.17 180)
 			(layer "F.Fab")
@@
 			)
 		)
-		(property "Value" "10kΩ"
+		(property "Value" "10k"
 			(at 0 1.17 0)
 			(layer "F.Fab")
@@
 			)
 		)
-		(property "Value" "100K"
+		(property "Value" "100k"
 			(at 0 1.17 127.235)
 			(layer "F.Fab")
@@
 			)
 		)
-		(property "Value" "100K"
+		(property "Value" "100k"
 			(at 0 1.17 127.235)
 			(layer "F.Fab")
@@
 			)
 		)
-		(property "Value" "10kΩ"
+		(property "Value" "10k"
 			(at 0 1.17 0)
 			(layer "F.Fab")
@@
 			)
 		)
-		(property "Value" "0.1µF"
+		(property "Value" "0.1uF"
 			(at 0 1.16 90)
 			(layer "F.Fab")
@@
 			)
 		)
-		(property "Value" "0.1µF"
+		(property "Value" "0.1uF"
 			(at 0 1.16 90)
 			(layer "F.Fab")
@@
 			)
 		)
-		(property "Value" "10kΩ"
+		(property "Value" "10k"
 			(at 0 1.17 90)
 			(layer "F.Fab")
@@
 			)
 		)
-		(property "Value" "0.1µF 25V"
+		(property "Value" "0.1uF 25V"
 			(at 0 1.16 0)
 			(layer "F.Fab")
@@
 			)
 		)
-		(property "Value" "10µF"
+		(property "Value" "10uF"
 			(at 0 1.43 0)
 			(layer "F.Fab")
@@
 			)
 		)
-		(property "Value" "100K"
+		(property "Value" "100k"
 			(at 0 1.17 0)
 			(layer "F.Fab")
@@
 			)
 		)
-		(property "Value" "20kΩ"
+		(property "Value" "20k"
 			(at 0 1.17 0)
 			(layer "F.Fab")
@@
 			)
 		)
-		(property "Value" "2.2µF"
+		(property "Value" "2.2uF"
 			(at 0 -1.43 0)
 			(layer "B.Fab")
@@
 			)
 		)
-		(property "Value" "10µF"
+		(property "Value" "10uF"
 			(at 0 -1.43 0)
 			(layer "B.Fab")
