File: hardware/boards/osc-sg90-m007/osc-sg90-m007.kicad_sch (KiCad schematic)
At the start: 32 parts, among them J1 TTL, J2 Motor, J3 PROG, J4 POT, Q1 MCMNP2065A-TP, Q2 MCMNP2065A-TP, U1 CH32M007E8U7

Commit message: hw: add osc-sg90-m007 renders to readme
Parts:
- C1, C3: value 10µF -> 10uF
- C2, C8: value 0.1µF -> 0.1uF
- C4: value 2.2µF -> 2.2uF
- C5: value 0.1µF 25V -> 0.1uF 25V
- R1, R2, R5, R6: value 100K -> 100k
- R11: value 4.7kΩ -> 4.7k
- R12, R4, R8: value 10kΩ -> 10k
- R13: value 33Ω -> 33
- R3, R7: value 20kΩ -> 20k
Changed lines of the file:
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@@
 			)
 		)
-		(property "Value" "10kΩ"
+		(property "Value" "10k"
 			(at 235.712 100.584 0)
 			(show_name no)
@@
 			)
 		)
-		(property "Value" "100K"
+		(property "Value" "100k"
 			(at 107.188 117.856 0)
 			(show_name no)
@@
 			)
 		)
-		(property "Value" "10kΩ"
+		(property "Value" "10k"
 			(at 143.256 112.268 0)
 			(show_name no)
@@
 			)
 		)
-		(property "Value" "2.2µF"
+		(property "Value" "2.2uF"
 			(at 60.198 43.688 0)
 			(show_name no)
@@
 			)
 		)
-		(property "Value" "100K"
+		(property "Value" "100k"
 			(at 107.696 93.472 0)
 			(show_name no)
@@
 			)
 		)
-		(property "Value" "10µF"
+		(property "Value" "10uF"
 			(at 22.606 97.79 0)
 			(show_name no)
@@
 			)
 		)
-		(property "Value" "100K"
+		(property "Value" "100k"
 			(at 36.068 119.126 0)
 			(show_name no)
@@
 			)
 		)
-		(property "Value" "0.1µF"
+		(property "Value" "0.1uF"
 			(at 194.77 115.03 0)
 			(show_name no)
@@
 			)
 		)
-		(property "Value" "20kΩ"
+		(property "Value" "20k"
 			(at 146.05 105.156 90)
 			(show_name no)
@@
 			)
 		)
-		(property "Value" "33Ω"
+		(property "Value" "33"
 			(at 243.078 34.798 0)
 			(show_name no)
@@
 			)
 		)
-		(property "Value" "0.1µF"
+		(property "Value" "0.1uF"
 			(at 23.114 44.704 0)
 			(show_name no)
@@
 			)
 		)
-		(property "Value" "4.7kΩ"
+		(property "Value" "4.7k"
 			(at 196.088 99.822 0)
 			(show_name no)
@@
 			)
 		)
-		(property "Value" "20kΩ"
+		(property "Value" "20k"
 			(at 74.93 106.426 90)
 			(show_name no)
@@
 			)
 		)
-		(property "Value" "100K"
+		(property "Value" "100k"
 			(at 36.576 94.742 0)
 			(show_name no)
@@
 			)
 		)
-		(property "Value" "10kΩ"
+		(property "Value" "10k"
 			(at 72.136 113.538 0)
 			(show_name no)
@@
 			)
 		)
-		(property "Value" "10µF"
+		(property "Value" "10uF"
 			(at 35.56 45.212 0)
 			(show_name no)
@@
 			)
 		)
-		(property "Value" "0.1µF 25V"
+		(property "Value" "0.1uF 25V"
 			(at 72.39 44.4562 0)
 			(show_name no)
