File: hardware/boards/osc-dev-v006/MCU.kicad_sch (KiCad schematic)
At the start: 7 parts, among them J4 PIN-2-3P, U3 CH32V006F8P6

Commit message: hw: osc-dev-v006 rev-c mcu pinout rewire
Connections:
- net DBG is gone; now on net EN: U3.13 (PC3)
- net ISNS+ is gone; now on net ENCB: U3.6 (PA2)
- net VSNS is gone; now on net ENCA: U3.5 (PA1)
- net EN: no longer U3.8 (PD0)
- net ENCA: no longer U3.20 (PD3)
- net ENCB: no longer U3.1 (PD4)
- net OPN2: no longer U3.4 (PA4)
- net RX: no longer U3.11 (PC1)
- net TX_EN renamed SCL
- new net OPA_N: U3.8 (PD0)
- new net OPA_OUT: U3.1 (PD4)
- new net OPA_P: U3.20 (PD3)
- new net SDA: U3.11 (PC1)
- new net nRST: U3.4 (PD7)
Changed lines of the file:
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@@
+	(wire
+		(pts
+			(xy 63.5 53.34) (xy 71.12 53.34)
+		)
+		(stroke
+			(width 0)
+			(type default)
+		)
+	)
 	(wire
 		(pts
@@
 		(pts
 			(xy 38.1 50.8) (xy 38.1 52.07)
-		)
-		(stroke
-			(width 0)
-			(type default)
-		)
-	)
-	(wire
-		(pts
-			(xy 64.77 53.34) (xy 71.12 53.34)
 		)
 		(stroke
@@
 		)
 	)
-	(label "OPN2"
-		(at 64.77 53.34 180)
+	(label "nRST"
+		(at 63.5 53.34 180)
 		(effects
 			(font
@@
 		)
 	)
-	(hierarchical_label "VSNS"
-		(shape input)
-		(at 71.12 55.88 180)
+	(hierarchical_label "ENCB"
+		(shape output)
+		(at 71.12 58.42 180)
 		(effects
 			(font
@@
 		)
 	)
+	(hierarchical_label "SCL"
+		(shape output)
+		(at 104.14 66.04 0)
+		(effects
+			(font
+				(size 1.27 1.27)
+			)
+			(justify left)
+		)
+	)
+	(hierarchical_label "OPA_N"
+		(shape input)
+		(at 71.12 63.5 180)
+		(effects
+			(font
+				(size 1.27 1.27)
+			)
+			(justify right)
+		)
+	)
 	(hierarchical_label "VSNB"
 		(shape input)
@@
 		)
 	)
-	(hierarchical_label "RX"
-		(shape input)
-		(at 104.14 68.58 0)
-		(effects
-			(font
-				(size 1.27 1.27)
-			)
-			(justify left)
-		)
-	)
 	(hierarchical_label "STAT"
 		(shape output)
@@
 		)
 	)
-	(hierarchical_label "ENCA"
+	(hierarchical_label "EN"
+		(shape output)
+		(at 104.14 63.5 0)
+		(effects
+			(font
+				(size 1.27 1.27)
+			)
+			(justify left)
+		)
+	)
+	(hierarchical_label "OPA_P"
 		(shape input)
 		(at 104.14 45.72 0)
-		(effects
-			(font
-				(size 1.27 1.27)
-			)
-			(justify left)
-		)
-	)
-	(hierarchical_label "STAT"
-		(shape output)
-		(at 104.14 53.34 0)
 		(effects
 			(font
@@
 		)
 	)
-	(hierarchical_label "EN"
-		(shape output)
-		(at 71.12 63.5 180)
-		(effects
-			(font
-				(size 1.27 1.27)
-			)
-			(justify right)
-		)
-	)
-	(hierarchical_label "ISNS+"
-		(shape input)
-		(at 71.12 58.42 180)
-		(effects
-			(font
-				(size 1.27 1.27)
-			)
-			(justify right)
+	(hierarchical_label "STAT"
+		(shape output)
+		(at 104.14 53.34 0)
+		(effects
+			(font
+				(size 1.27 1.27)
+			)
+			(justify left)
 		)
 	)
@@
 		)
 	)
-	(hierarchical_label "ENCB"
+	(hierarchical_label "OPA_OUT"
 		(shape input)
 		(at 71.12 45.72 180)
@@
 		)
 	)
-	(hierarchical_label "DBG"
-		(shape output)
-		(at 104.14 63.5 0)
-		(effects
-			(font
-				(size 1.27 1.27)
-			)
-			(justify left)
-		)
-	)
-	(hierarchical_label "TX_EN"
-		(shape output)
-		(at 104.14 66.04 0)
-		(effects
-			(font
-				(size 1.27 1.27)
-			)
-			(justify left)
+	(hierarchical_label "ENCA"
+		(shape output)
+		(at 71.12 55.88 180)
+		(effects
+			(font
+				(size 1.27 1.27)
+			)
+			(justify right)
 		)
 	)
@@
 		(shape input)
 		(at 104.14 48.26 0)
+		(effects
+			(font
+				(size 1.27 1.27)
+			)
+			(justify left)
+		)
+	)
+	(hierarchical_label "SDA"
+		(shape output)
+		(at 104.14 68.58 0)
 		(effects
 			(font
@@
 		)
 		(pin "8"
+			(alternate "OPN1")
 		)
 		(pin "5"
-			(alternate "A1")
+			(alternate "T2C2_5")
 		)
 		(pin "9"
@@
 		)
 		(pin "6"
-			(alternate "OPP0")
+			(alternate "T2C3_5")
 		)
 		(pin "2"
@@
 		)
 		(pin "4"
-			(alternate "OPN2")
+			(alternate "RST")
 		)
 		(pin "1"
-			(alternate "A7")
+			(alternate "OPO0")
 		)
 		(pin "11"
-			(alternate "RX_3")
+			(alternate "SDA")
 		)
 		(pin "15"
@@
 		)
 		(pin "12"
+			(alternate "SCL")
 		)
 		(pin "13"
@@
 		)
 		(pin "20"
-			(alternate "A4")
+			(alternate "OPP2")
 		)
 		(pin "17"
