File: hardware/boards/osc-dev-v006/osc-dev-v006.kicad_sch (KiCad schematic)
At the start: 4 parts

Commit message: hw: osc-dev-v006 rev-c mcu pinout rewire
Changed lines of the file:
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@@
 			)
 		)
-		(pin "ENCA" input
+		(pin "ENCA" output
 			(at 115.57 142.24 180)
 			(effects
@@
 			)
 		)
-		(pin "ENCB" input
+		(pin "ENCB" output
 			(at 115.57 144.78 180)
 			(effects
