File: hardware/boards/osc-dev-v006/MOTOR_DRIVER.kicad_sch (KiCad schematic)
At the start: 8 parts, among them J4 MOT, U3 DRV8212PDSGR

Commit message: board: osc-dev-v006 rev 2a (#107)
Parts:
- removed C6: 100nF, Capacitor_SMD:C_0603_1608Metric_Pad1.08x0.95mm_HandSolder, symbol Device:C
- removed FB1: 600Ω@100MHz, Inductor_SMD:L_0603_1608Metric_Pad1.05x0.95mm_HandSolder, symbol Device:FerriteBead_Small
- added Ch1: 100nF, Capacitor_SMD:C_0603_1608Metric_Pad1.08x0.95mm_HandSolder, symbol Device:C
- added Ch4: 10uF, Capacitor_SMD:C_0805_2012Metric_Pad1.18x1.45mm_HandSolder, symbol Device:C
- added Rh2: 0R, Resistor_SMD:R_0603_1608Metric_Pad0.98x0.95mm_HandSolder, symbol Device:R
- added TP3: IN1, TestPoint:TestPoint_Pad_D1.0mm, symbol Connector:TestPoint_Small
- added TP4: IN2, TestPoint:TestPoint_Pad_D1.0mm, symbol Connector:TestPoint_Small
- Ch3: renamed from C8; value 10µF -> 10uF
- Ch5: renamed from C9; value 100µF -> 100uF
- J4: LCSC (none) -> C492401; MFPN (none) -> 2.54-1*2P
- Rh1: renamed from R14; MFPN FRC0805F1002TS -> FRC0603F1002TS
- U3: footprint Package_SON:Texas_DSG0008A_WSON-8-1EP_2x2mm_P0.5mm_EP0.9x1.6mm -> Package_SON:Texas_DSG0008A_WSON-8-1EP_2x2mm_P0.5mm_EP0.9x1.6mm_ThermalVias; JLC Type Extended -> (none)
- renumbered C7 to Ch2
Connections:
- net +3V3: now also Rh2.1
- net +3V3_DRV: now also Ch1.1, Rh2.2
- net DRV_IN1: now also TP3.1
- net DRV_IN2: now also TP4.1
- net GND: now also Ch1.2, Ch4.2
- net VSYS: now also Ch4.1
Other:
- note added: "Decoupling and bulk"
- note added: "Motor driver"
- note added: "Motor header"
- note removed: "DRIVER IC"
- note removed: "LOGIC SUPPLY"
- note removed: "Motor Header"
- moved on the sheet: Ch2, Ch3, Ch5
