File: hardware/boards/osc-dev-v006/SENSORS.kicad_sch (KiCad schematic)
At the start: 46 parts, among them J5 POS, J6 ENC, J7 NTC

Commit message: hw: v006 lcsc fields track rev-2a order substitutions
Parts:
- C13, Cd1: LCSC C24452 -> C14663; MFPN CL21B104KCFNNNE -> CC0603KRX7R9BB104
- Cc1, Cc2: LCSC C1653 -> C105620; MFPN CL21C220JBANNNC -> CC0603JRNPO9BN220
- Cc6: LCSC C1653 -> C105620; MFPN CC0805JRNPO9BN330 -> CC0603JRNPO9BN220
- Cin1, Cv1, Cv2: LCSC C14858 -> C14665; MFPN CC0805JRNPO9BN101 -> CC0603JRNPO9BN101
- Ck1: LCSC C14858 -> C14665; MFPN CL21C102JBCNNNC -> CC0603JRNPO9BN101
- Rk1, Rk2: LCSC C21189 -> C95177; MFPN FRC0805F0000TS -> RC0603JR-070RL
Changed lines of the file:
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@@
 			)
 		)
-		(property "Datasheet" "https://www.lcsc.com/product-detail/C21189.html"
+		(property "Datasheet" "https://www.lcsc.com/product-detail/C95177.html"
 			(at 57.15 64.77 0)
 			(hide yes)
@@
 			)
 		)
-		(property "Description" "Resistor"
+		(property "Description" "0Ω jumper 100mW 0603"
 			(at 57.15 64.77 0)
 			(hide yes)
@@
 			)
 		)
-		(property "LCSC" "C21189"
+		(property "LCSC" "C95177"
 			(at 57.15 62.484 0)
 			(hide yes)
@@
 			)
 		)
-		(property "MFPN" "FRC0805F0000TS"
+		(property "MFPN" "RC0603JR-070RL"
 			(at 57.15 62.484 0)
 			(hide yes)
@@
 			)
 		)
-		(property "Datasheet" "https://www.lcsc.com/product-detail/C1653.html"
+		(property "Datasheet" "https://www.lcsc.com/product-detail/C105620.html"
 			(at 161.29 67.31 0)
 			(hide yes)
@@
 			)
 		)
-		(property "Description" "Unpolarized capacitor"
+		(property "Description" "22pF ±5% 50V NP0 0603"
 			(at 161.29 67.31 0)
 			(hide yes)
@@
 			)
 		)
-		(property "LCSC" "C1653"
+		(property "LCSC" "C105620"
 			(at 165.1 66.0399 0)
 			(hide yes)
@@
 			)
 		)
-		(property "MFPN" "CL21C220JBANNNC"
+		(property "MFPN" "CC0603JRNPO9BN220"
 			(at 165.1 66.0399 0)
 			(hide yes)
@@
 			)
 		)
-		(property "Datasheet" "https://www.lcsc.com/product-detail/C14858.html"
+		(property "Datasheet" "https://www.lcsc.com/product-detail/C14665.html"
 			(at 105.95 90.18 0)
 			(hide yes)
@@
 			)
 		)
-		(property "Description" "Unpolarized capacitor"
+		(property "Description" "100pF ±5% 50V NP0 0603"
 			(at 105.95 90.18 0)
 			(hide yes)
@@
 			)
 		)
-		(property "LCSC" "C14858"
+		(property "LCSC" "C14665"
 			(at 65.278 111.76 0)
 			(hide yes)
@@
 			)
 		)
-		(property "MFPN" "CC0805JRNPO9BN101"
+		(property "MFPN" "CC0603JRNPO9BN101"
 			(at 65.278 111.76 0)
 			(hide yes)
@@
 			)
 		)
-		(property "Datasheet" "https://www.lcsc.com/product-detail/C21189.html"
+		(property "Datasheet" "https://www.lcsc.com/product-detail/C95177.html"
 			(at 57.15 49.53 0)
 			(hide yes)
@@
 			)
 		)
-		(property "Description" "Resistor"
+		(property "Description" "0Ω jumper 100mW 0603"
 			(at 57.15 49.53 0)
 			(hide yes)
@@
 			)
 		)
-		(property "LCSC" "C21189"
+		(property "LCSC" "C95177"
 			(at 57.15 47.244 0)
 			(hide yes)
@@
 			)
 		)
-		(property "MFPN" "FRC0805F0000TS"
+		(property "MFPN" "RC0603JR-070RL"
 			(at 57.15 47.244 0)
 			(hide yes)
@@
 			)
 		)
-		(property "Datasheet" "https://www.lcsc.com/product-detail/C24452.html"
+		(property "Datasheet" "https://www.lcsc.com/product-detail/C14663.html"
 			(at 127.72 138.99 0)
 			(hide yes)
@@
 			)
 		)
-		(property "Description" "Unpolarized capacitor"
+		(property "Description" "100nF ±10% 50V X7R 0603"
 			(at 127.72 138.99 0)
 			(hide yes)
@@
 			)
 		)
-		(property "LCSC" "C24452"
+		(property "LCSC" "C14663"
 			(at 115.316 117.856 0)
 			(hide yes)
@@
 			)
 		)
-		(property "MFPN" "CL21B104KCFNNNE"
+		(property "MFPN" "CC0603KRX7R9BB104"
 			(at 115.316 117.856 0)
 			(hide yes)
@@
 			)
 		)
-		(property "Datasheet" "https://www.lcsc.com/product-detail/C14858.html"
+		(property "Datasheet" "https://www.lcsc.com/product-detail/C14665.html"
 			(at 62.23 57.15 0)
 			(hide yes)
@@
 			)
 		)
-		(property "Description" "Unpolarized capacitor"
+		(property "Description" "100pF ±5% 50V NP0 0603"
 			(at 62.23 57.15 0)
 			(hide yes)
@@
 			)
 		)
-		(property "MFPN" "CL21C102JBCNNNC"
+		(property "MFPN" "CC0603JRNPO9BN101"
 			(at 62.23 57.15 0)
 			(hide yes)
@@
 			)
 		)
-		(property "LCSC" "C14858"
+		(property "LCSC" "C14665"
 			(at 62.23 57.15 0)
 			(hide yes)
@@
 			)
 		)
-		(property "Datasheet" "https://www.lcsc.com/product-detail/C24452.html"
+		(property "Datasheet" "https://www.lcsc.com/product-detail/C14663.html"
 			(at 96.52 58.42 0)
 			(hide yes)
@@
 			)
 		)
-		(property "Description" "Unpolarized capacitor"
+		(property "Description" "100nF ±10% 50V X7R 0603"
 			(at 96.52 58.42 0)
 			(hide yes)
@@
 			)
 		)
-		(property "LCSC" "C24452"
+		(property "LCSC" "C14663"
 			(at 98.044 55.626 0)
 			(hide yes)
@@
 			)
 		)
-		(property "MFPN" "CL21B104KCFNNNE"
+		(property "MFPN" "CC0603KRX7R9BB104"
 			(at 98.044 55.626 0)
 			(hide yes)
@@
 			)
 		)
-		(property "Datasheet" "https://www.lcsc.com/product-detail/C14858.html"
+		(property "Datasheet" "https://www.lcsc.com/product-detail/C14665.html"
 			(at 177.8 57.15 0)
 			(hide yes)
@@
 			)
 		)
-		(property "Description" "Unpolarized capacitor"
+		(property "Description" "100pF ±5% 50V NP0 0603"
 			(at 177.8 57.15 0)
 			(hide yes)
@@
 			)
 		)
-		(property "LCSC" "C14858"
+		(property "LCSC" "C14665"
 			(at 181.61 55.8799 0)
 			(hide yes)
@@
 			)
 		)
-		(property "MFPN" "CC0805JRNPO9BN101"
+		(property "MFPN" "CC0603JRNPO9BN101"
 			(at 181.61 55.8799 0)
 			(hide yes)
@@
 			)
 		)
-		(property "Datasheet" "https://www.lcsc.com/product-detail/C1653.html"
+		(property "Datasheet" "https://www.lcsc.com/product-detail/C105620.html"
 			(at 161.29 46.99 0)
 			(hide yes)
@@
 			)
 		)
-		(property "Description" "Unpolarized capacitor"
+		(property "Description" "22pF ±5% 50V NP0 0603"
 			(at 161.29 46.99 0)
 			(hide yes)
@@
 			)
 		)
-		(property "LCSC" "C1653"
+		(property "LCSC" "C105620"
 			(at 165.1 45.7199 0)
 			(hide yes)
@@
 			)
 		)
-		(property "MFPN" "CL21C220JBANNNC"
+		(property "MFPN" "CC0603JRNPO9BN220"
 			(at 165.1 45.7199 0)
 			(hide yes)
@@
 			)
 		)
-		(property "Datasheet" "https://www.lcsc.com/product-detail/C14858.html"
+		(property "Datasheet" "https://www.lcsc.com/product-detail/C14665.html"
 			(at 67.85 90.18 0)
 			(hide yes)
@@
 			)
 		)
-		(property "Description" "Unpolarized capacitor"
+		(property "Description" "100pF ±5% 50V NP0 0603"
 			(at 67.85 90.18 0)
 			(hide yes)
@@
 			)
 		)
-		(property "LCSC" "C14858"
+		(property "LCSC" "C14665"
 			(at 27.178 111.76 0)
 			(hide yes)
@@
 			)
 		)
-		(property "MFPN" "CC0805JRNPO9BN101"
+		(property "MFPN" "CC0603JRNPO9BN101"
 			(at 27.178 111.76 0)
 			(hide yes)
@@
 			)
 		)
-		(property "Datasheet" "https://www.lcsc.com/product-detail/C1653.html"
+		(property "Datasheet" "https://www.lcsc.com/product-detail/C105620.html"
 			(at 121.92 182.88 0)
 			(hide yes)
@@
 			)
 		)
-		(property "Description" "Unpolarized capacitor"
+		(property "Description" "22pF ±5% 50V NP0 0603"
 			(at 121.92 182.88 0)
 			(hide yes)
@@
 			)
 		)
-		(property "LCSC" "C1653"
+		(property "LCSC" "C105620"
 			(at 125.73 181.6099 0)
 			(hide yes)
@@
 			)
 		)
-		(property "MFPN" "CC0805JRNPO9BN330"
+		(property "MFPN" "CC0603JRNPO9BN220"
 			(at 125.73 181.6099 0)
 			(hide yes)

Commit message: board: osc-dev-v006 rev 2a (#107)
Parts:
- removed Cc5: 10pF, Capacitor_SMD:C_0603_1608Metric_Pad1.08x0.95mm_HandSolder, symbol Device:C
- removed Cc6: 22pF, Capacitor_SMD:C_0603_1608Metric_Pad1.08x0.95mm_HandSolder, symbol Device:C
- removed Ck2: 470pF, Capacitor_SMD:C_0603_1608Metric_Pad1.08x0.95mm_HandSolder, symbol Device:C
- removed R22: 10K, Resistor_SMD:R_0603_1608Metric_Pad0.98x0.95mm_HandSolder, symbol Device:R
- removed RS2: 60m, Resistor_SMD:R_1206_3216Metric, symbol Device:R
- removed RS3: 22m, Resistor_SMD:R_1206_3216Metric, symbol Device:R
- removed Rg3: 300, Resistor_SMD:R_0603_1608Metric_Pad0.98x0.95mm_HandSolder, symbol Device:R
- removed Rg4, Rk5: 100, Resistor_SMD:R_0603_1608Metric_Pad0.98x0.95mm_HandSolder, symbol Device:R
- removed Rk3: 20, Resistor_SMD:R_0603_1608Metric_Pad0.98x0.95mm_HandSolder, symbol Device:R
- removed Rk4: 47, Resistor_SMD:R_0603_1608Metric_Pad0.98x0.95mm_HandSolder, symbol Device:R
- removed TP3: GND, TestPoint:TestPoint_Pad_D1.0mm, symbol Connector:TestPoint_Small
- added Ca2, Cb2: 100nF, Capacitor_SMD:C_0603_1608Metric_Pad1.08x0.95mm_HandSolder, symbol Device:C
- added Cb1: 10uF, Capacitor_SMD:C_0805_2012Metric_Pad1.18x1.45mm_HandSolder, symbol Device:C
- added Co1: 22pF, Capacitor_SMD:C_0603_1608Metric_Pad1.08x0.95mm_HandSolder, symbol Device:C
- added Cv3: 100pF, Capacitor_SMD:C_0603_1608Metric_Pad1.08x0.95mm_HandSolder, symbol Device:C
- added J11: Conn_01x06, shared:Flex_Landing_1x06_P1.0mm, symbol Connector_Generic:Conn_01x06
- added Ra2: 4K7, Resistor_SMD:R_0603_1608Metric_Pad0.98x0.95mm_HandSolder, symbol Device:R
- added Rb1: 430, Resistor_SMD:R_0603_1608Metric_Pad0.98x0.95mm_HandSolder, symbol Device:R
- added Rb2: 100, Resistor_SMD:R_0603_1608Metric_Pad0.98x0.95mm_HandSolder, symbol Device:R
- added Rn1: 10K, Resistor_SMD:R_0603_1608Metric_Pad0.98x0.95mm_HandSolder, symbol Device:R
- added Rv5: 6K4, Resistor_SMD:R_0603_1608Metric_Pad0.98x0.95mm_HandSolder, symbol Device:R
- added Rv6: 1K6, Resistor_SMD:R_0603_1608Metric_Pad0.98x0.95mm_HandSolder, symbol Device:R
- added TP5: VA, TestPoint:TestPoint_Pad_D1.0mm, symbol Connector:TestPoint_Small
- added TP6: VB, TestPoint:TestPoint_Pad_D1.0mm, symbol Connector:TestPoint_Small
- added TP7: VS, TestPoint:TestPoint_Pad_D1.0mm, symbol Connector:TestPoint_Small
- added TP8: VP1, TestPoint:TestPoint_Pad_D1.0mm, symbol Connector:TestPoint_Small
- added TP9: VP2, TestPoint:TestPoint_Pad_D1.0mm, symbol Connector:TestPoint_Small
- Cc3, Cc4: value 47pF -> 22pF; LCSC C1671 -> C105620; MFPN CC0805JRNPO9BN470 -> CC0603JRNPO9BN220
- Ck1: JLC_Basic yes -> (none)
- J5: footprint Connector_PinHeader_2.54mm:PinHeader_1x03_P2.54mm_Vertical -> Connector_PinHeader_2.54mm:PinHeader_1x04_P2.54mm_Vertical; symbol Connector_Generic:Conn_01x03 -> Connector_Generic:Conn_01x04; LCSC C49257 -> (none); MFPN 2.54-1*3P -> 2.54-1*4P
- J7: footprint Connector_PinHeader_2.54mm:PinHeader_1x02_P2.54mm_Vertical -> Connector_PinHeader_2.54mm:PinHeader_1x03_P2.54mm_Vertical; symbol Connector_Generic:Conn_01x02 -> Connector_Generic:Conn_01x03; LCSC C492401 -> C49257; MFPN 2.54-1*2P -> 2.54-1*3P
- Ra1: renamed from R21; MFPN FRC0805F4701TS -> FRC0603F4701TS
- Rd1: MFPN FRC0805F1001TS -> AR03DTC1601
- Rd2: MFPN FRC0805F1800TS -> AR03DTC3000
- Rd3: MFPN FRC0805F1500TS -> AR03DTC3000
- Rf1, Rf2: MFPN ARG03DTC7501 -> AR03DTC6401N
- Rg1, Rg2: MFPN ARG03DTC4990 -> AR03DTCX4300
- Rk1, Rk2: value 0 -> 0R
- Rs1: renamed from RS1; value 33m -> 60m; footprint Resistor_SMD:R_1206_3216Metric -> Resistor_SMD:R_1206_3216Metric_Pad1.30x1.75mm_HandSolder; LCSC C49164942 -> C49164944; MFPN JER1206F1R033 -> JER1206F1R060
- Rv1, Rv3: value 20K -> 6K4; LCSC C319764 -> C374580; MFPN ARG03DTC2002 -> AR03DTC6401N
- Rv2, Rv4: value 10K -> 1K6; LCSC C319937 -> C374557; MFPN ARG02DTC1002 -> AR03DTC1601
- TH1: value 10kΩ 3950K -> 10K/3950; MFPN SDNT2012X103F3950FTF -> CMFA103F3950
- TP1: now left out of the parts list
- TP2: value GND -> OPA; now left out of the parts list
- renumbered C13 to Ca1, Cin1 to Ci1
Connections:
- net +3V3: now also J7.2 (Pin_2), J11.2 (Pin_2), Rb1.1, Rn1.1
- net ENCA: now also J11.3 (Pin_3)
- net ENCB: now also J11.4 (Pin_4)
- net GND: now also J7.3 (Pin_3), Ca2.2, Cb1.2, Cb2.2, Co1.2, Cv3.2, J11.1 (Pin_1), J11.6 (Pin_6), Rb2.2, Rv6.2; no longer Cv1.2, Cv2.2, J7.2 (Pin_2), Rv2.2, Rv4.2, TP2.1
- net OPA_OUT: now also TP2.1, Co1.1
- net VNTC_EXT: now also J11.5 (Pin_5)
- net VNTC_INT: now also Rn1.2
- net VSNA: now also TP5.1
- net VSNB: now also TP6.1
- net POT renamed POS1
- net VNTC renamed VPOS2_NTC
- net VPOS2_NTC: now also Ca2.1, Ra2.1, TP9.1
- net VPOS renamed VPOS1
- net VPOS1: now also TP8.1
- new net POS2: J5.4 (Pin_4), Ra2.2
- new net VB: Cb1.1, Cb2.1, Cv1.2, Cv2.2, Rb1.2, Rb2.1, Rv2.2, Rv4.2
- new net VSNS: Cv3.1, Rv5.2, Rv6.1, TP7.1
- new net VSYS: Rv5.1
- no-connect marks 18 -> 0
Other:
- note added: "Current sense shunt"
- note added: "NTC temperature"
- note added: "OPA difference amplifier"
- note added: "Sensor connectors"
- note added: "Servo pot"
- note added: "Terminal and supply sense"
- note removed: "BENCH SWAP KIT"
- note removed: "CONNECTORS"
- note removed: "CURRENT SHUNT"
- note removed: "MOTOR BEMF"
- note removed: "NTC TEMP"
- note removed: "OPA BIAS"
- note removed: "SERVO POT"
- note removed: "TEST POINTS"
- moved on the sheet: Ca1, Cc1, Cc2, Cc3, Cc4, Ci1, Ck1, J6, JP2, NT1, NT2, Ra1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
